File: driver_card_4234520/4234520.kicad_pcb (KiCad board)
At the start: 2 copper layers, 152.4 x 107.2 mm, 39 parts, among them J1 Bus_ISA_8bit, J2 DC62_Female, U1 74LS74, U10 74LS155, U11 74LS02, U12 74LS09, U13 74LS244, U14 74LS244, U15 74LS21, U16 74LS244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

Commit message: make library paths relative convert to 4 layer pcb add gnd and 5v planes symbol cleanup ERC zero errors!
Routing:
- added copper zone on In2.Cu, net /5V
- added copper zone on In1.Cu, net /GND
Other:
- copper layers 2 -> 4
Changed lines of the file:
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@@
   (layers
     (0 "F.Cu" signal)
+    (1 "In1.Cu" signal)
+    (2 "In2.Cu" signal)
     (31 "B.Cu" signal)
     (32 "B.Adhes" user "B.Adhesive")
@@
       (layer "F.Mask" (type "Top Solder Mask") (thickness 0.01))
       (layer "F.Cu" (type "copper") (thickness 0.035))
-      (layer "dielectric 1" (type "core") (thickness 1.51) (material "FR4") (epsilon_r 4.5) (loss_tangent 0.02))
+      (layer "dielectric 1" (type "prepreg") (thickness 0.1) (material "FR4") (epsilon_r 4.5) (loss_tangent 0.02))
+      (layer "In1.Cu" (type "copper") (thickness 0.035))
+      (layer "dielectric 2" (type "core") (thickness 1.24) (material "FR4") (epsilon_r 4.5) (loss_tangent 0.02))
+      (layer "In2.Cu" (type "copper") (thickness 0.035))
+      (layer "dielectric 3" (type "prepreg") (thickness 0.1) (material "FR4") (epsilon_r 4.5) (loss_tangent 0.02))
       (layer "B.Cu" (type "copper") (thickness 0.035))
       (layer "B.Mask" (type "Bottom Solder Mask") (thickness 0.01))
@@
   (via (at 142.24 74.93) (size 1.65) (drill 1.4) (layers "F.Cu" "B.Cu") (free) (net 102))
   (via (at 142.24 82.55) (size 1.65) (drill 1.4) (layers "F.Cu" "B.Cu") (free) (net 103))
+  (zone (net 1) (net_name "/GND") (layer "In1.Cu") (hatch edge 0.5)
+    (connect_pads (clearance 0.5))
+    (min_thickness 0.25) (filled_areas_thickness no)
+    (fill (thermal_gap 0.5) (thermal_bridge_width 0.5))
+    (polygon
+      (pts
+        (xy 10.16 10.16)
+        (xy 162.56 10.16)
+        (xy 162.56 109.22)
+        (xy 10.16 109.22)
+      )
+    )
+  )
+  (zone (net 3) (net_name "/5V") (layer "In2.Cu") (hatch edge 0.5)
+    (priority 1)
+    (connect_pads (clearance 0.5))
+    (min_thickness 0.25) (filled_areas_thickness no)
+    (fill (thermal_gap 0.5) (thermal_bridge_width 0.5))
+    (polygon
+      (pts
+        (xy 10.16 10.16)
+        (xy 162.56 10.16)
+        (xy 162.56 109.22)
+        (xy 10.16 109.22)
+      )
+    )
+  )
 )
